File: hw-thingcell.kicad_sch (KiCad schematic)
At the start: 95 parts, among them J1 Conn_01x02_Pin, J2 Conn_01x08_Pin, J3 Conn_01x08_Pin, J4 USB4510-03-1-A, J5 GSM_ANT, J6 GNSS_ANT, J7 SIM8060-6-0-14-00-A, Q2 PMBT3904235, Q3 PMBT3904235, Q4 PMBT3904235, U1 AP62301WU-7, U2 AP62301WU-7, U3 ESP32-S2-SOLO, U4 SIM868, U5 CH340C, Y1 32.768k

Commit message: Sch reviewed
Parts:
- added R11, R9: NC, Resistor_SMD:R_0402_1005Metric, symbol Device:R
- added TP15: VDD_EXT, TestPoint:TestPoint_Pad_D1.0mm, symbol Connector:TestPoint
- added TP5: VBUS, TestPoint:TestPoint_Pad_D1.0mm, symbol Connector:TestPoint
- renumbered D3 to D2, D5 to D3, D6 to D4, D7 to D5, D8 to D6, D9 to D7, D10 to D8, J3 to J2, J4 to J3, J2 to J4, Q3 to Q1, Q4 to Q2, Q2 to Q3, R14 to R10, R11 to R12, R23 to R13, R24 to R14, R12 to R15, R13 to R16, R15 to R17, R16 to R18, R17 to R19, R18 to R20, R19 to R21, R20 to R22, R21 to R23, R22 to R24, R10 to R6, R8 to R7, R9 to R8, TP9 to TP10, TP10 to TP11, TP11 to TP12, TP12 to TP13, TP13 to TP14, TP14 to TP16, TP5 to TP6, TP6 to TP7, TP7 to TP8, TP8 to TP9
Connections:
- net EXT7 is gone; now on net D7/SS: J2.5 (Pin_5)
- net EXT8 is gone; now on net D8: J2.6 (Pin_6)
- net EXT9 is gone; now on net D9/S_DET: J2.7 (Pin_7)
- net GPIO1 is gone; now on net D3: U3.20 (GPIO12/TOUCH12/ADC2_CH1/FSPICLK/FSPIIO6)
- net GPIO2 is gone; now on net D4/SCK: U3.21 (GPIO13/TOUCH13/ADC2_CH2/FSPIQ/FSPIIO7)
- net GPIO3 is gone; now on net D5/MISO: U3.22 (GPIO14/TOUCH14/ADC2_CH3/FSPIWP/FSPIDQS)
- net I2C_SCL is gone; now on net D2/SDA: U3.19 (GPIO11/TOUCH11/ADC2_CH0/FSPID/FSPIIO5)
- net I2C_SDA is gone; now on net D1/SCL: U3.18 (GPIO10/TOUCH10/ADC1_CH9/FSPICS0/FSPIIO4)
- net +3V3: now also J4.3 (Pin_3), R11.1, R9.1; no longer J4.4 (Pin_4)
- net +4V: no longer J4.3 (Pin_3)
- net PK_CTL: now also U3.17 (GPIO9/TOUCH9/ADC1_CH8/FSPIHD); no longer U3.10 (GPIO17/U1TXD/ADC2_CH6/DAC_1)
- net VBUS: now also J4.2 (Pin_2), TP5.1
- net VIN: now also J4.4 (Pin_4); no longer J4.2 (Pin_2)
- net D7/SS: now reaches U3.24 (SPIIO4/GPIO33/FSPIHD)
- net D8: now reaches U3.25 (SPIIO5/GPIO34/FSPICS0)
- net D9/S_DET: now reaches U3.28 (SPIIO6/GPIO35/FSPID)
- net at U4.40 (VDD_EXT): now also TP15.1
- net EXT1 renamed D1/SCL
- net D1/SCL: now also R9.2
- net EXT2 renamed D2/SDA
- net D2/SDA: now also R11.2
- net EXT3 renamed D3
- net EXT4 renamed D4/SCK
- net EXT5 renamed D5/MISO
- net EXT6 renamed D6/MOSI
- net D6/MOSI: now also U3.10 (GPIO17/U1TXD/ADC2_CH6/DAC_1)
- net SIM_DET: no longer names the net of U4.14 (SIM1_DET)
- net SIM_DET: no longer U3.17 (GPIO9/TOUCH9/ADC1_CH8/FSPIHD)
- no-connect marks 51 -> 49
Other:
- note added: "Reference projects: https://github.com/Xinyuan-LilyGO/ LilyGo-T-Call-SIM800 https://www.waveshare.com/w/upload/ 6/65/Pico-SIM868-GSM-GPRS-GNSS-Schematic.pdf"
- note added: "TODO Review ESP GPIOS Review testpoints Add LEDs"
- note removed: "2 filas de conectores de expansión Posibles placas de expansión: BAT, RELAY+HiLink, x3RELAY+HiLink 2.54 mm Alimentación: entradas: Vin, GND salidas: Vin, 4V, 3V3, GND GPIOS: relé (hasta 3), LEDs?, SPI, I2C, touch? Shield detect?"
- note removed: "Reference projects: https://github.com/Xinyuan-LilyGO/LilyGo-T-Call-SIM800 https://www.waveshare.com/w/upload/6/65/Pico-SIM868-GSM-GPRS-GNSS-Schematic.pdf"
- note removed: "TODO Supply and relay diodes? Relay? Relay diode? V for relay? (VIN/4V/3V3) Expansion connector (I2C con pullups o GPIOs? interfaces?) Review USB-C connections VDD_EXT SIM not connected to anything Review ESP GPIOS Revisar testpoints Axadir LEDs"
- moved on the sheet: D1, J1, J2, J3, J4, Q1, Q2, R10, R13, R14, R6, TP6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
