File: hw-thingcell.kicad_sch (KiCad schematic)
At the start: 99 parts, among them J1 Conn_01x02_Pin, J2 Conn_01x08_Pin, J3 USB4510-03-1-A, J4 Conn_01x08_Pin, J5 GSM_ANT, J6 GNSS_ANT, J7 SIM8060-6-0-14-00-A, Q1 PMBT3904235, Q2 PMBT3904235, Q3 PMBT3904235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

Commit message: First placement
Other:
- note added: "TODO Review ESP GPIOS Review testpoints Add LEDs Add button?"
- note removed: "TODO Review ESP GPIOS Review testpoints Add LEDs"
Changed lines of the file:
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@@
     (effects (font (size 1.27 1.27)) (justify left bottom))
   )
-  (text "TODO\nReview ESP GPIOS\nReview testpoints\nAdd LEDs\n" (at 228.6 144.78 0)
+  (text "TODO\nReview ESP GPIOS\nReview testpoints\nAdd LEDs\nAdd button?"
+    (at 228.6 144.78 0)
     (effects (font (size 1.27 1.27)) (justify left bottom))
   )

Commit message: First placement
Parts:
- added J1: Conn_01x02_Pin, Connector_PinSocket_2.54mm:PinSocket_1x02_P2.54mm_Vertical, symbol Connector:Conn_01x02_Pin
- J2: renamed from J1; footprint Connector_PinHeader_2.54mm:PinHeader_1x02_P2.54mm_Vertical -> Connector_PinSocket_2.54mm:PinSocket_1x02_P2.54mm_Vertical
- renumbered J2 to J3, J3 to J4, J4 to J5, J5 to J6, J6 to J7, J7 to J8
Connections:
- net GND: now also J1.2 (Pin_2)
- net VIN: now also J1.1 (Pin_1)

Commit message: Routed all components
Connections:
- net D1/SCL: now also U3.29 (SPIIO7/GPIO36/FSPICLK); no longer U3.18 (GPIO10/TOUCH10/ADC1_CH9/FSPICS0/FSPIIO4)
- net D2/SDA: now also U3.28 (SPIIO6/GPIO35/FSPID); no longer U3.19 (GPIO11/TOUCH11/ADC2_CH0/FSPID/FSPIIO5)
- net D3: now also U3.30 (SPIDQS/GPIO37/FSPIQ); no longer U3.20 (GPIO12/TOUCH12/ADC2_CH1/FSPICLK/FSPIIO6)
- net D4/SCK: now also U3.4 (GPIO4/TOUCH4/ADC1_CH3); no longer U3.21 (GPIO13/TOUCH13/ADC2_CH2/FSPIQ/FSPIIO7)
- net D5/MISO: now also U3.5 (GPIO5/TOUCH5/ADC1_CH4); no longer U3.22 (GPIO14/TOUCH14/ADC2_CH3/FSPIWP/FSPIDQS)
- net D6/MOSI: now also U3.6 (GPIO6/TOUCH6/ADC1_CH5); no longer U3.10 (GPIO17/U1TXD/ADC2_CH6/DAC_1)
- net D7/SS: now also U3.7 (GPIO7/TOUCH7/ADC1_CH6); no longer U3.24 (SPIIO4/GPIO33/FSPIHD)
- net D8: now also U3.10 (GPIO17/U1TXD/ADC2_CH6/DAC_1); no longer U3.25 (SPIIO5/GPIO34/FSPICS0)
- net D9/S_DET: now also U3.12 (GPIO8/TOUCH8/ADC1_CH7); no longer U3.28 (SPIIO6/GPIO35/FSPID)
- net ESP_CTS: now also U3.19 (GPIO11/TOUCH11/ADC2_CH0/FSPID/FSPIIO5); no longer U3.38 (GPIO2/TOUCH2/ADC1_CH1)
- net ESP_IO32: now also U3.17 (GPIO9/TOUCH9/ADC1_CH8/FSPIHD); no longer U3.6 (GPIO6/TOUCH6/ADC1_CH5)
- net ESP_IO33: now also U3.18 (GPIO10/TOUCH10/ADC1_CH9/FSPICS0/FSPIIO4); no longer U3.7 (GPIO7/TOUCH7/ADC1_CH6)
- net ESP_IO34: now also U3.15 (GPIO3/TOUCH3/ADC1_CH2); no longer U3.12 (GPIO8/TOUCH8/ADC1_CH7)
- net ESP_RTS: now also U3.20 (GPIO12/TOUCH12/ADC2_CH1/FSPICLK/FSPIIO6); no longer U3.15 (GPIO3/TOUCH3/ADC1_CH2)
- net ESP_RXD: now also U3.22 (GPIO14/TOUCH14/ADC2_CH3/FSPIWP/FSPIDQS); no longer U3.4 (GPIO4/TOUCH4/ADC1_CH3)
- net ESP_TXD: now also U3.21 (GPIO13/TOUCH13/ADC2_CH2/FSPIQ/FSPIIO7); no longer U3.5 (GPIO5/TOUCH5/ADC1_CH4)
- net PK_CTL: now also U3.25 (SPIIO5/GPIO34/FSPICS0); no longer U3.17 (GPIO9/TOUCH9/ADC1_CH8/FSPIHD)
Other:
- moved on the sheet: TP10, TP11, TP12, TP13

Commit message: Work in texts and graphics
Parts:
- removed TP4: 5V, TestPoint:TestPoint_Pad_D1.0mm, symbol Connector:TestPoint
Connections:
- net +5V is gone; now on net VBUS: J4.A9 (VBUS_2)
- net +3V3: now also J5.2 (Pin_2); no longer J5.3 (Pin_3)
- net VBUS: now also J5.3 (Pin_3); no longer J5.2 (Pin_2)
Other:
- moved on the sheet: TP5, TP6

Commit message: Final revision
Parts:
- added C22: 100n, Capacitor_SMD:C_0402_1005Metric, symbol Device:C
Connections:
- net +3V3: no longer U5.4 (V3)
- net GND: now also C22.2
- new net: C22.1, U5.4 (V3)
- no-connect marks 49 -> 50
Other:
- note removed: "TODO Review ESP GPIOS Review testpoints Add LEDs Add button?"
Changed lines of the file:
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@@
   (junction (at 81.28 167.64) (diameter 0) (color 0 0 0 0)
   )
-  (junction (at 176.53 129.54) (diameter 0) (color 0 0 0 0)
-  )
   (junction (at 229.87 19.05) (diameter 0) (color 0 0 0 0)
   )
@@
   (no_connect (at 184.15 80.01))
   (no_connect (at 184.15 85.09))
+  (no_connect (at 168.91 152.4))
   (no_connect (at 46.99 45.72))
   (no_connect (at 153.67 44.45))
@@
     (stroke (width 0) (type default))
   )
-  (wire (pts (xy 176.53 129.54) (xy 179.07 129.54))
-    (stroke (width 0) (type default))
-  )
   (wire (pts (xy 184.15 36.83) (xy 201.93 36.83))
     (stroke (width 0) (type default))
@@
     (stroke (width 0) (type default))
   )
+  (wire (pts (xy 189.23 129.54) (xy 179.07 129.54))
+    (stroke (width 0) (type default))
+  )
   (wire (pts (xy 33.02 87.63) (xy 38.1 87.63))
     (stroke (width 0) (type default))
@@
     (effects (font (size 1.27 1.27)) (justify left bottom))
   )
-  (text "TODO\nReview ESP GPIOS\nReview testpoints\nAdd LEDs\nAdd button?"
-    (at 228.6 144.78 0)
-    (effects (font (size 1.27 1.27)) (justify left bottom))
-  )
   (text "Expansion port" (at 101.6 170.18 0)
     (effects (font (size 2 2) (thickness 0.4) bold) (justify left bottom))
@@
     )
   )
+  (symbol (lib_id "Device:C") (at 193.04 129.54 90) (unit 1)
+    (in_bom yes) (on_board yes) (dnp no)
+    (property "Reference" "C22" (at 196.85 127 90)
+      (effects (font (size 1.27 1.27)))
+    )
+    (property "Value" "100n" (at 189.23 127 90)
+      (effects (font (size 1.27 1.27)))
+    )
+    (property "Footprint" "Capacitor_SMD:C_0402_1005Metric" (at 196.85 128.5748 0)
+      (effects (font (size 1.27 1.27)) hide)
+    )
+    (property "Datasheet" "~" (at 193.04 129.54 0)
+      (effects (font (size 1.27 1.27)) hide)
+    )
+    (pin "1")
+    (pin "2")
+    (instances
+      (project "hw-thingcell"
+        (path "/b864757b-52bc-4794-ab53-eb54b6429a77"
+          (reference "C22") (unit 1)
+        )
+      )
+    )
+  )
   (symbol (lib_id "Device:R") (at 72.39 151.13 0) (unit 1)
     (in_bom yes) (on_board yes) (dnp no)
@@
         )
       )
+    )
+  )
+  (symbol (lib_id "power:GND") (at 196.85 129.54 90) (unit 1)
+    (in_bom yes) (on_board yes) (dnp no)
+    (property "Reference" "#PWR012" (at 203.2 129.54 0)
+      (effects (font (size 1.27 1.27)) hide)
+    )
+    (property "Value" "GND" (at 201.93 129.54 90)
+      (effects (font (size 1.27 1.27)))
+    )
+    (property "Footprint" "" (at 196.85 129.54 0)
+      (effects (font (size 1.27 1.27)) hide)
+    )
+    (property "Datasheet" "" (at 196.85 129.54 0)
+      (effects (font (size 1.27 1.27)) hide)
+    )
+    (pin "1")
+    (instances
+      (project "hw-thingcell"
+        (path "/b864757b-52bc-4794-ab53-eb54b6429a77"
+          (reference "#PWR012") (unit 1)
+        )
+      )
